File: PCBs/GDEnvSensorGW_1_15/GDEnvSensorGW_1_15.sch (EAGLE design)
At the start: 42 parts, among them CN1 1X4FPC0.5, Q1 NPN, Q2 NPN, U1 3.3V, U3 RFM69HCW, X1 ZX62D-B-5PA8, X2 SMA

Commit message: Version 1.15 of GW board
Parts:
- removed C15: 10uF, SparkFun-Capacitors:10UF10V10%(0805)
- added C5: .1uF, SparkFun-Capacitors:10UF10V10%(0805)
- added IC2: MCP4017T, SamacSys_Parts:MCP4017T-503E_LT
- added MIC6122: MIC6122, SamacSys_Parts:MIC6211YM5-TR
- added R10: 22k, adafruit:R-US_R0805
- added R15: 13.3K, adafruit:R-US_R0805
- added R16, R17: 10k, adafruit:R-US_R0805
- added R9: 100K 1%, adafruit:R-US_R0805
- added U4: LTR-329, SamacSys_Parts:LTR-329ALS-01
- R8: value 102k -> 10K 1%
Connections:
- removed net N$10: R11.2, R12.1, R8.1
- new net N$12: IC2.W, R10.1
- new net N$2: MIC6122.IN+, R15.1, R8.2
- new net N$6: C5.2, IC2.B, MIC6122.OUT, R11.2, R12.1
- new net N$7: MIC6122.IN-, R10.2, R9.1
- net 12V: now also MIC6122.V+, R15.2, R9.2; no longer C15.1, R8.2
- net 3.3V: now also 12V.EN, 12V.IN, C4.2, FB1.P$1, IC2.VDD, R16.2, R17.2, U4.VDD
- net GND: now also C5.1, IC2.VSS, MIC6122.V-, R8.1, U4.GND; no longer C15.2
- net SCL: now also IC2.SCL, R16.1, U4.SCL
- net SDA: now also IC2.SDA, R17.1, U4.SDA
- net VIN_PROT: no longer 12V.EN, 12V.IN, C4.2, FB1.P$1
Other:
- moved on the sheet: 12V, C2, C3, C4, D5, FB1, LED1, R1, R11, R12, R2, R3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
